File: C264Cart.kicad_sch (KiCad schematic)
At the start: 13 parts, among them U1 27C040, U3 264-Exp-Port

Commit message: updated to SMD components (except EPROM)
Parts:
- C1: footprint Capacitor_THT:C_Disc_D6.0mm_W2.5mm_P5.00mm -> Capacitor_SMD:C_0603_1608Metric
- D1, D2: footprint Diode_THT:D_DO-35_SOD27_P7.62mm_Horizontal -> Diode_SMD:D_SOD-323
- JP1, JP2, JP3, JP4, JP5, JP6: footprint C264Cart:Jumper3_Solder -> Jumper:SolderJumper-3_P1.3mm_Open_RoundedPad1.0x1.5mm
- JP7: footprint C264Cart:Jumper3_Solder -> Jumper:SolderJumper-2_P1.3mm_Open_RoundedPad1.0x1.5mm
- R1: footprint Resistor_THT:R_Axial_DIN0207_L6.3mm_D2.5mm_P7.62mm_Horizontal -> Resistor_SMD:R_0603_1608Metric
