File: plus4cart.kicad_sch (KiCad schematic)
At the start: 13 parts, among them U1 27C040, U3 264-Exp-Port

Commit message: updated schema/pcb metadata
Other:
- company: www.hackup.net -> maciaszek.net
- title: C264Cart -> plus4cart
Changed lines of the file:
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@@
 	(paper "A4")
 	(title_block
-		(title "C264Cart")
-		(date "2023-11-28")
+		(title "plus4cart")
+		(date "2026-05-03")
 		(rev "1")
-		(company "www.hackup.net")
+		(company "maciaszek.net")
 		(comment 1 "Creative Commons Attribution-NonCommercial-ShareAlike 4.0 International License.")
 		(comment 2 "This work is licensed under a")
+		(comment 3 "Based on C264Cart made by hackup.net")
 	)
 	(junction
